Commit message: Added rviz visualization of real robot

File: quad_simulator/a1_description/xacro/leg.xacro (robot description, xacro)
@@ -88,8 +88,8 @@
         </link>
         <joint name="${hipJointName}" type="revolute">
-            <origin rpy="0 ${PI/2.0} 0" xyz="0 ${thigh_offset*mirror} 0"/>
+            <origin rpy="0 0 0" xyz="0 ${thigh_offset*mirror} 0"/>
             <parent link="hip${suffix}"/>
             <child link="upper${suffix}"/>
-            <axis xyz="0 -1 0"/>
+            <axis xyz="0 1 0"/>
             <dynamics damping="${damping}" friction="${friction}"/>
             <limit effort="${thigh_torque_max}" velocity="${thigh_velocity_max}" lower="${thigh_min*PI/180.0}" upper="${thigh_max*PI/180.0}"/>
@@ -116,5 +116,5 @@
         </link>
         <joint name="${kneeJointName}" type="revolute">
-            <origin rpy="0 ${-PI} 0" xyz="0 0 ${-thigh_length}"/>
+            <origin rpy="0 0 0" xyz="0 0 ${-thigh_length}"/>
             <parent link="upper${suffix}"/>
             <child link="lower${suffix}"/>

File: quad_simulator/a1_description/xacro/robot.xacro (robot description, xacro)
@@ -107,21 +107,21 @@
     </link>
     <!--FL-->
-    <xacro:leg suffix="0" mirror="1" mirror_dae="True" front_hind="1" front_hind_dae="True"
-               hipJointName="0" kneeJointName="1" abductionJointName="8">
+    <xacro:leg suffix="1" mirror="1" mirror_dae="True" front_hind="1" front_hind_dae="True"
+               hipJointName="4" kneeJointName="5" abductionJointName="3">
         <origin rpy="0 0 0" xyz="${leg_offset_x} ${leg_offset_y} 0"/>
     </xacro:leg>
     <!--RL-->
-    <xacro:leg suffix="1" mirror="1" mirror_dae="True" front_hind="-1" front_hind_dae="False"
-               hipJointName="2" kneeJointName="3" abductionJointName="9">
+    <xacro:leg suffix="3" mirror="1" mirror_dae="True" front_hind="-1" front_hind_dae="False"
+               hipJointName="10" kneeJointName="11" abductionJointName="9">
         <origin rpy="0 0 0" xyz="${-leg_offset_x} ${leg_offset_y} 0"/>
     </xacro:leg>
     <!--FR-->
-    <xacro:leg suffix="2" mirror="-1" mirror_dae="False" front_hind="1" front_hind_dae="True"
-               hipJointName="4" kneeJointName="5" abductionJointName="10">
+    <xacro:leg suffix="0" mirror="-1" mirror_dae="False" front_hind="1" front_hind_dae="True"
+               hipJointName="1" kneeJointName="2" abductionJointName="0">
         <origin rpy="0 0 0" xyz="${leg_offset_x} ${-leg_offset_y} 0"/>
     </xacro:leg>
     <!--RR-->
-    <xacro:leg suffix="3" mirror="-1" mirror_dae="False" front_hind="-1" front_hind_dae="False"
-               hipJointName="6" kneeJointName="7" abductionJointName="11">
+    <xacro:leg suffix="2" mirror="-1" mirror_dae="False" front_hind="-1" front_hind_dae="False"
+               hipJointName="7" kneeJointName="8" abductionJointName="6">
         <origin rpy="0 0 0" xyz="${-leg_offset_x} ${-leg_offset_y} 0"/>
     </xacro:leg>

Commit message: Returned original xacro description. Implemented joint transforms from robot to quad

File: quad_simulator/a1_description/xacro/leg.xacro (robot description, xacro)
@@ -88,8 +88,8 @@
         </link>
         <joint name="${hipJointName}" type="revolute">
-            <origin rpy="0 0 0" xyz="0 ${thigh_offset*mirror} 0"/>
+            <origin rpy="0 ${PI/2.0} 0" xyz="0 ${thigh_offset*mirror} 0"/>
             <parent link="hip${suffix}"/>
             <child link="upper${suffix}"/>
-            <axis xyz="0 1 0"/>
+            <axis xyz="0 -1 0"/>
             <dynamics damping="${damping}" friction="${friction}"/>
             <limit effort="${thigh_torque_max}" velocity="${thigh_velocity_max}" lower="${thigh_min*PI/180.0}" upper="${thigh_max*PI/180.0}"/>
@@ -116,5 +116,5 @@
         </link>
         <joint name="${kneeJointName}" type="revolute">
-            <origin rpy="0 0 0" xyz="0 0 ${-thigh_length}"/>
+            <origin rpy="0 ${-PI} 0" xyz="0 0 ${-thigh_length}"/>
             <parent link="upper${suffix}"/>
             <child link="lower${suffix}"/>

File: quad_simulator/a1_description/xacro/robot.xacro (robot description, xacro)
@@ -8,5 +8,5 @@
     <xacro:property name="rolloverProtection" value="false"/>
     <!-- Debug mode will hung up the robot, use "true" or "false" to switch it. -->
-    <xacro:if value="$(arg DEBUG)">
+    <!-- <xacro:if value="$(arg DEBUG)">
         <link name="world"/>
         <joint name="base_static_joint" type="fixed">
@@ -15,5 +15,5 @@
             <child link="body"/>
         </joint>
-    </xacro:if>
+    </xacro:if>  -->
     <link name="body">
         <visual>
@@ -107,21 +107,21 @@
     </link>
     <!--FL-->
-    <xacro:leg suffix="1" mirror="1" mirror_dae="True" front_hind="1" front_hind_dae="True"
-               hipJointName="4" kneeJointName="5" abductionJointName="3">
+    <xacro:leg suffix="0" mirror="1" mirror_dae="True" front_hind="1" front_hind_dae="True"
+               hipJointName="0" kneeJointName="1" abductionJointName="8">
         <origin rpy="0 0 0" xyz="${leg_offset_x} ${leg_offset_y} 0"/>
     </xacro:leg>
     <!--RL-->
-    <xacro:leg suffix="3" mirror="1" mirror_dae="True" front_hind="-1" front_hind_dae="False"
-               hipJointName="10" kneeJointName="11" abductionJointName="9">
+    <xacro:leg suffix="1" mirror="1" mirror_dae="True" front_hind="-1" front_hind_dae="False"
+               hipJointName="2" kneeJointName="3" abductionJointName="9">
         <origin rpy="0 0 0" xyz="${-leg_offset_x} ${leg_offset_y} 0"/>
     </xacro:leg>
     <!--FR-->
-    <xacro:leg suffix="0" mirror="-1" mirror_dae="False" front_hind="1" front_hind_dae="True"
-               hipJointName="1" kneeJointName="2" abductionJointName="0">
+    <xacro:leg suffix="2" mirror="-1" mirror_dae="False" front_hind="1" front_hind_dae="True"
+               hipJointName="4" kneeJointName="5" abductionJointName="10">
         <origin rpy="0 0 0" xyz="${leg_offset_x} ${-leg_offset_y} 0"/>
     </xacro:leg>
     <!--RR-->
-    <xacro:leg suffix="2" mirror="-1" mirror_dae="False" front_hind="-1" front_hind_dae="False"
-               hipJointName="7" kneeJointName="8" abductionJointName="6">
+    <xacro:leg suffix="3" mirror="-1" mirror_dae="False" front_hind="-1" front_hind_dae="False"
+               hipJointName="6" kneeJointName="7" abductionJointName="11">
         <origin rpy="0 0 0" xyz="${-leg_offset_x} ${-leg_offset_y} 0"/>
     </xacro:leg>
