Commit message: kinda added realsense

File: quad_simulator/a1_description/urdf/a1.urdf (robot description, URDF)
Before this commit: robot a1_description, 23 links, 22 joints
Links:
- link hip0: mass 0.696 -> 0.591
- link hip1: mass 0.696 -> 0.591
- link hip2: mass 0.696 -> 0.591
- link hip3: mass 0.696 -> 0.591
- link lower0: mass 0.166 -> 0.135862; geometry collision box size=0.213 0.016 0.016; visual mesh filename=package://a1_description/meshes/calf.dae scale=1 1 1
- link lower1: mass 0.166 -> 0.135862; geometry collision box size=0.213 0.016 0.016; visual mesh filename=package://a1_description/meshes/calf.dae scale=1 1 1
- link lower2: mass 0.166 -> 0.135862; geometry collision box size=0.213 0.016 0.016; visual mesh filename=package://a1_description/meshes/calf.dae scale=1 1 1
- link lower3: mass 0.166 -> 0.135862; geometry collision box size=0.213 0.016 0.016; visual mesh filename=package://a1_description/meshes/calf.dae scale=1 1 1
- link trunk: mass 6.0 -> 5.204; geometry collision box size=0.3762 0.0935 0.114; visual mesh filename=package://a1_description/meshes/trunk.dae scale=1 1 1
- link upper0: mass 1.013 -> 0.92; geometry collision box size=0.213 0.0245 0.034; visual mesh filename=package://a1_description/meshes/thigh.dae scale=1 1 1
- link upper1: mass 1.013 -> 0.92; geometry collision box size=0.213 0.0245 0.034; visual mesh filename=package://a1_description/meshes/thigh.dae scale=1 1 1
- link upper2: mass 1.013 -> 0.92; geometry collision box size=0.213 0.0245 0.034; visual mesh filename=package://a1_description/meshes/thigh_mirror.dae scale=1 1 1
- link upper3: mass 1.013 -> 0.92; geometry collision box size=0.213 0.0245 0.034; visual mesh filename=package://a1_description/meshes/thigh_mirror.dae scale=1 1 1
Joints:
- joint 0: limit lower=-6.28318530718 upper=6.28318530718 effort=33.5 velocity=21 -> lower=-0.0119729586686811 upper=0.07855726963226478 effort=23.7 velocity=30.1; origin xyz=0 0.0838 0 rpy=0 1.57079632679 0 -> xyz=0 0.08 0 rpy=0 1.5707963267948966 0
- joint 1: limit lower=-6.28318530718 upper=6.28318530718 effort=33.5 velocity=21 -> lower=-0.049183378321200205 upper=-0.015498523757709647 effort=35.55 velocity=20.06; origin xyz=0 0 -0.2 rpy=0 -3.14159265359 0 -> xyz=0 0 -0.213 rpy=0 -3.141592653589793 0
- joint 10: limit lower=-0.802851455917 upper=0.802851455917 effort=33.5 velocity=21 -> lower=-0.015062191444711064 upper=0.015062191444711064 effort=23.7 velocity=30.1; origin xyz=0.1805 -0.047 0 rpy=0 0 0 -> xyz=0.1881 -0.04675 0 rpy=0 0 0
- joint 11: limit lower=-0.802851455917 upper=0.802851455917 effort=33.5 velocity=21 -> lower=-0.015062191444711064 upper=0.015062191444711064 effort=23.7 velocity=30.1; origin xyz=-0.1805 -0.047 0 rpy=0 0 0 -> xyz=-0.1881 -0.04675 0 rpy=0 0 0
- joint 2: limit lower=-6.28318530718 upper=6.28318530718 effort=33.5 velocity=21 -> lower=-0.0119729586686811 upper=0.07855726963226478 effort=23.7 velocity=30.1; origin xyz=0 0.0838 0 rpy=0 1.57079632679 0 -> xyz=0 0.08 0 rpy=0 1.5707963267948966 0
- joint 3: limit lower=-6.28318530718 upper=6.28318530718 effort=33.5 velocity=21 -> lower=-0.049183378321200205 upper=-0.015498523757709647 effort=35.55 velocity=20.06; origin xyz=0 0 -0.2 rpy=0 -3.14159265359 0 -> xyz=0 0 -0.213 rpy=0 -3.141592653589793 0
- joint 4: limit lower=-6.28318530718 upper=6.28318530718 effort=33.5 velocity=21 -> lower=-0.0119729586686811 upper=0.07855726963226478 effort=23.7 velocity=30.1; origin xyz=0 -0.0838 0 rpy=0 1.57079632679 0 -> xyz=0 -0.08 0 rpy=0 1.5707963267948966 0
- joint 5: limit lower=-6.28318530718 upper=6.28318530718 effort=33.5 velocity=21 -> lower=-0.049183378321200205 upper=-0.015498523757709647 effort=35.55 velocity=20.06; origin xyz=0 0 -0.2 rpy=0 -3.14159265359 0 -> xyz=0 0 -0.213 rpy=0 -3.141592653589793 0
- joint 6: limit lower=-6.28318530718 upper=6.28318530718 effort=33.5 velocity=21 -> lower=-0.0119729586686811 upper=0.07855726963226478 effort=23.7 velocity=30.1; origin xyz=0 -0.0838 0 rpy=0 1.57079632679 0 -> xyz=0 -0.08 0 rpy=0 1.5707963267948966 0
- joint 7: limit lower=-6.28318530718 upper=6.28318530718 effort=33.5 velocity=21 -> lower=-0.049183378321200205 upper=-0.015498523757709647 effort=35.55 velocity=20.06; origin xyz=0 0 -0.2 rpy=0 -3.14159265359 0 -> xyz=0 0 -0.213 rpy=0 -3.141592653589793 0
- joint 8: limit lower=-0.802851455917 upper=0.802851455917 effort=33.5 velocity=21 -> lower=-0.015062191444711064 upper=0.015062191444711064 effort=23.7 velocity=30.1; origin xyz=0.1805 0.047 0 rpy=0 0 0 -> xyz=0.1881 0.04675 0 rpy=0 0 0
- joint 9: limit lower=-0.802851455917 upper=0.802851455917 effort=33.5 velocity=21 -> lower=-0.015062191444711064 upper=0.015062191444711064 effort=23.7 velocity=30.1; origin xyz=-0.1805 0.047 0 rpy=0 0 0 -> xyz=-0.1881 0.04675 0 rpy=0 0 0
- joint hip0_fixed: origin xyz=0 0.081 0 rpy=0 0 0 -> xyz=0 0.096 0 rpy=0 0 0
- joint hip1_fixed: origin xyz=0 0.081 0 rpy=0 0 0 -> xyz=0 0.096 0 rpy=0 0 0
- joint hip2_fixed: origin xyz=0 -0.081 0 rpy=0 0 0 -> xyz=0 -0.096 0 rpy=0 0 0
- joint hip3_fixed: origin xyz=0 -0.081 0 rpy=0 0 0 -> xyz=0 -0.096 0 rpy=0 0 0
- joint jtoe0: origin xyz=0 0 -0.2 rpy=0 0 0 -> xyz=0 0 -0.213 rpy=0 0 0
- joint jtoe1: origin xyz=0 0 -0.2 rpy=0 0 0 -> xyz=0 0 -0.213 rpy=0 0 0
- joint jtoe2: origin xyz=0 0 -0.2 rpy=0 0 0 -> xyz=0 0 -0.213 rpy=0 0 0
- joint jtoe3: origin xyz=0 0 -0.2 rpy=0 0 0 -> xyz=0 0 -0.213 rpy=0 0 0

File: quad_simulator/a1_description/xacro/const.xacro (robot description, xacro)
@@ -1,10 +1,10 @@
 <?xml version="1.0"?>
-<robot name="a1_description" xmlns:xacro="http://www.ros.org/wiki/xacro">
+<robot xmlns:xacro="http://www.ros.org/wiki/xacro">
     <!-- Constants for robot dimensions -->
     <xacro:property name="PI" value="3.1415926535897931"/>
     <xacro:property name="stick_mass" value="0.00001"/>
     <!-- simplified collision value -->
-    <xacro:property name="trunk_width" value="0.194"/>
-    <xacro:property name="trunk_length" value="0.267"/>
+    <xacro:property name="trunk_width" value="0.0935"/>
+    <xacro:property name="trunk_length" value="0.3762"/>
     <xacro:property name="trunk_height" value="0.114"/>
     <xacro:property name="hip_radius" value="0.046"/>
@@ -19,84 +19,127 @@
     <xacro:property name="stick_radius" value="0.01"/>
     <xacro:property name="stick_length" value="0.2"/>
+    <!-- kinematic value -->
+    <xacro:property name="thigh_offset" value="0.08"/>
+    <xacro:property name="thigh_length" value="0.213"/>
+    <xacro:property name="calf_length" value="0.213"/>
+    <!-- leg offset from trunk center value -->
+    <xacro:property name="leg_offset_x" value="0.1881"/>
+    <xacro:property name="leg_offset_y" value="0.04675"/>
+    <!-- <xacro:property name="trunk_offset_z" value="0.01675"/> -->
+    <xacro:property name="hip_offset" value="0.08"/>
+    <!-- offset of link and rotor locations (left front) -->
+    <xacro:property name="hip_offset_x" value="0.1881"/>
+    <xacro:property name="hip_offset_y" value="0.04675"/>
+    <xacro:property name="hip_offset_z" value="0.0"/>
+    <xacro:property name="hip_rotor_offset_x" value="0.11215"/>
+    <xacro:property name="hip_rotor_offset_y" value="0.04675"/>
+    <xacro:property name="hip_rotor_offset_z" value="0.0"/>
+    <xacro:property name="thigh_offset_x" value="0"/>
+    <xacro:property name="thigh_offset_y" value="0.08"/>
+    <xacro:property name="thigh_offset_z" value="0.0"/>
+    <xacro:property name="thigh_rotor_offset_x" value="0.0"/>
+    <xacro:property name="thigh_rotor_offset_y" value="-0.00015"/>
+    <xacro:property name="thigh_rotor_offset_z" value="0.0"/>
+    <xacro:property name="calf_offset_x" value="0.0"/>
+    <xacro:property name="calf_offset_y" value="0.0"/>
+    <xacro:property name="calf_offset_z" value="-0.213"/>
+    <xacro:property name="calf_rotor_offset_x" value="0.0"/>
+    <xacro:property name="calf_rotor_offset_y" value="-0.03235"/>
+    <xacro:property name="calf_rotor_offset_z" value="0.0"/>
+    <!-- joint limits -->
+    <xacro:property name="damping" value="0.01"/>
+    <xacro:property name="friction" value="0.2"/>
+    <xacro:property name="hip_position_max" value="0.863"/>
+    <xacro:property name="hip_position_min" value="-0.863"/>
+    <xacro:property name="hip_velocity_max" value="30.1"/>
+    <xacro:property name="hip_torque_max" value="23.7"/>
+    <xacro:property name="thigh_position_max" value="4.501"/>
+    <xacro:property name="thigh_position_min" value="-0.686"/>
+    <xacro:property name="thigh_velocity_max" value="30.1"/>
+    <xacro:property name="thigh_torque_max" value="23.7"/>
+    <xacro:property name="calf_position_max" value="-0.888"/>
+    <xacro:property name="calf_position_min" value="-2.818"/>
+    <xacro:property name="calf_velocity_max" value="20.06"/>
+    <xacro:property name="calf_torque_max" value="35.55"/>
+    <!-- dynamics inertial value        total 12.84kg -->
+    <!-- trunk -->
+    <xacro:property name="trunk_mass" value="5.204"/>
+    <xacro:property name="trunk_com_x" value="0.0223"/>
+    <xacro:property name="trunk_com_y" value="0.002"/>
+    <xacro:property name="trunk_com_z" value="-0.0005"/>
+    <xacro:property name="trunk_ixx" value="0.0168128557"/>
+    <xacro:property name="trunk_ixy" value="-0.0002296769"/>
+    <xacro:property name="trunk_ixz" value="-0.0002945293"/>
+    <xacro:property name="trunk_iyy" value="0.063009565"/>
+    <xacro:property name="trunk_iyz" value="-0.0000418731"/>
+    <xacro:property name="trunk_izz" value="0.0716547275"/>
+    <!-- hip (left front) -->
+    <xacro:property name="hip_mass" value="0.591"/>
+    <xacro:property name="hip_com_x" value="-0.005657"/>
+    <xacro:property name="hip_com_y" value="-0.008752"/>
+    <xacro:property name="hip_com_z" value="-0.000102"/>
+    <xacro:property name="hip_ixx" value="0.000334008405"/>
+    <xacro:property name="hip_ixy" value="-0.000010826066"/>
+    <xacro:property name="hip_ixz" value="0.000001290732"/>
+    <xacro:property name="hip_iyy" value="0.000619101213"/>
+    <xacro:property name="hip_iyz" value="0.000001643194"/>
+    <xacro:property name="hip_izz" value="0.00040057614"/>
+    <xacro:property name="hip_rotor_mass" value="0.089"/>
+    <xacro:property name="hip_rotor_com_x" value="0.0"/>
+    <xacro:property name="hip_rotor_com_y" value="0.0"/>
+    <xacro:property name="hip_rotor_com_z" value="0.0"/>
+    <xacro:property name="hip_rotor_ixx" value="0.000111842"/>
+    <xacro:property name="hip_rotor_ixy" value="0.0"/>
+    <xacro:property name="hip_rotor_ixz" value="0.0"/>
+    <xacro:property name="hip_rotor_iyy" value="0.000059647"/>
+    <xacro:property name="hip_rotor_iyz" value="0.0"/>
+    <xacro:property name="hip_rotor_izz" value="0.000059647"/>
+    <!-- thigh -->
+    <xacro:property name="thigh_mass" value="0.92"/>
+    <xacro:property name="thigh_com_x" value="-0.003342"/>
+    <xacro:property name="thigh_com_y" value="-0.018054"/>
+    <xacro:property name="thigh_com_z" value="-0.033451"/>
+    <xacro:property name="thigh_ixx" value="0.004431760472"/>
+    <xacro:property name="thigh_ixy" value="0.000057496807"/>
+    <xacro:property name="thigh_ixz" value="-0.000218457134"/>
+    <xacro:property name="thigh_iyy" value="0.004485671726"/>
+    <xacro:property name="thigh_iyz" value="0.000572001265"/>
+    <xacro:property name="thigh_izz" value="0.000740309489"/>
+    <xacro:property name="thigh_rotor_mass" value="0.089"/>
+    <xacro:property name="thigh_rotor_com_x" value="0.0"/>
+    <xacro:property name="thigh_rotor_com_y" value="0.0"/>
+    <xacro:property name="thigh_rotor_com_z" value="0.0"/>
+    <xacro:property name="thigh_rotor_ixx" value="0.000059647"/>
+    <xacro:property name="thigh_rotor_ixy" value="0.0"/>
+    <xacro:property name="thigh_rotor_ixz" value="0.0"/>
+    <xacro:property name="thigh_rotor_iyy" value="0.000111842"/>
+    <xacro:property name="thigh_rotor_iyz" value="0.0"/>
+    <xacro:property name="thigh_rotor_izz" value="0.000059647"/>
+    <!-- calf -->
+    <xacro:property name="calf_mass" value="0.135862"/>
+    <xacro:property name="calf_com_x" value="0.006197"/>
+    <xacro:property name="calf_com_y" value="0.001408"/>
+    <xacro:property name="calf_com_z" value="-0.116695"/>
+    <xacro:property name="calf_ixx" value="0.001088793059"/>
+    <xacro:property name="calf_ixy" value="-0.000000255679"/>
+    <xacro:property name="calf_ixz" value="0.000007117814"/>
+    <xacro:property name="calf_iyy" value="0.001100428748"/>
+    <xacro:property name="calf_iyz" value="0.000002077264"/>
+    <xacro:property name="calf_izz" value="0.000024787446"/>
+    <xacro:property name="calf_rotor_mass" value="0.089"/>
+    <xacro:property name="calf_rotor_com_x" value="0.0"/>
+    <xacro:property name="calf_rotor_com_y" value="0.0"/>
+    <xacro:property name="calf_rotor_com_z" value="0.0"/>
+    <xacro:property name="calf_rotor_ixx" value="0.000059647"/>
+    <xacro:property name="calf_rotor_ixy" value="0.0"/>
+    <xacro:property name="calf_rotor_ixz" value="0.0"/>
+    <xacro:property name="calf_rotor_iyy" value="0.000111842"/>
+    <xacro:property name="calf_rotor_iyz" value="0.0"/>
+    <xacro:property name="calf_rotor_izz" value="0.000059647"/>
+    <!-- foot -->
+    <xacro:property name="foot_mass" value="0.06"/>
     <xacro:property name="toe_friction" value="0.2"/>
     <xacro:property name="toe_lateral_friction" value="0.2"/>
     <xacro:property name="toe_stiffness" value="30000.0"/>
     <xacro:property name="toe_damping" value="1000.0"/>
-    <!-- kinematic value -->
-    <xacro:property name="thigh_offset" value="0.0838"/>
-    <xacro:property name="thigh_length" value="0.2"/>
-    <xacro:property name="calf_length" value="0.2"/>
-    <!-- leg offset from trunk center value -->
-    <xacro:property name="leg_offset_x" value="0.1805"/>
-    <xacro:property name="leg_offset_y" value="0.047"/>
-    <xacro:property name="trunk_offset_z" value="0.01675"/>
-    <xacro:property name="hip_offset" value="0.065"/>
-    <!-- joint limits -->
-    <xacro:property name="damping" value="0"/>
-    <xacro:property name="friction" value="0"/>
-    <!-- <xacro:property name="hip_max" value="46"/>
-    <xacro:property name="hip_min" value="-46"/> -->
-    <xacro:property name="hip_max" value="46"/>
-    <xacro:property name="hip_min" value="-46"/>
-    <xacro:property name="hip_velocity_max" value="21"/>
-    <xacro:property name="hip_torque_max" value="33.5"/>
-    <!-- <xacro:property name="thigh_max" value="240"/>
-    <xacro:property name="thigh_min" value="-60"/> -->
-    <xacro:property name="thigh_max" value="360"/>
-    <xacro:property name="thigh_min" value="-360"/>
-    <xacro:property name="thigh_velocity_max" value="21"/>
-    <xacro:property name="thigh_torque_max" value="33.5"/>
-    <!-- <xacro:property name="calf_max" value="-52.5"/>
-    <xacro:property name="calf_min" value="-154.5"/> -->
-    <xacro:property name="calf_max" value="360"/>
-    <xacro:property name="calf_min" value="-360"/>
-    <xacro:property name="calf_velocity_max" value="21"/>
-    <xacro:property name="calf_torque_max" value="33.5"/>
-    <!-- dynamics inertial value -->
-    <!-- trunk -->
-    <xacro:property name="trunk_mass" value="6.0"/>
-    <xacro:property name="trunk_com_x" value="0.0000"/>
-    <xacro:property name="trunk_com_y" value="0.0041"/>
-    <xacro:property name="trunk_com_z" value="-0.0005"/>
-    <xacro:property name="trunk_ixx" value="0.0158533"/>
-    <xacro:property name="trunk_ixy" value="-0.0000366"/>
-    <xacro:property name="trunk_ixz" value="-0.0000611"/>
-    <xacro:property name="trunk_iyy" value="0.0377999"/>
-    <xacro:property name="trunk_iyz" value="-0.0000275"/>
-    <xacro:property name="trunk_izz" value="0.0456542"/>
-    <!-- hip (left front) -->
-    <xacro:property name="hip_mass" value="0.696"/>
-    <xacro:property name="hip_com_x" value="-0.003311"/>
-    <xacro:property name="hip_com_y" value="0.000635"/>
-    <xacro:property name="hip_com_z" value="0.000031"/>
-    <xacro:property name="hip_ixx" value="0.000469246"/>
-    <xacro:property name="hip_ixy" value="-0.000009409"/>
-    <xacro:property name="hip_ixz" value="-0.000000342"/>
-    <xacro:property name="hip_iyy" value="0.000807490"/>
-    <xacro:property name="hip_iyz" value="-0.000000466"/>
-    <xacro:property name="hip_izz" value="0.000552929"/>
-    <!-- thigh -->
-    <xacro:property name="thigh_mass" value="1.013"/>
-    <xacro:property name="thigh_com_x" value="-0.003237"/>
-    <xacro:property name="thigh_com_y" value="-0.022327"/>
-    <xacro:property name="thigh_com_z" value="-0.027326"/>
-    <xacro:property name="thigh_ixx" value="0.005529065"/>
-    <xacro:property name="thigh_ixy" value="0.000004825"/>
-    <xacro:property name="thigh_ixz" value="0.000343869"/>
-    <xacro:property name="thigh_iyy" value="0.005139339"/>
-    <xacro:property name="thigh_iyz" value="0.000022448"/>
-    <xacro:property name="thigh_izz" value="0.001367788"/>
-    <!-- calf -->
-    <xacro:property name="calf_mass" value="0.166"/>
-    <xacro:property name="calf_com_x" value="0.006435"/>
-    <xacro:property name="calf_com_y" value="0.0"/>
-    <xacro:property name="calf_com_z" value="-0.107388"/>
-    <xacro:property name="calf_ixx" value="0.002997972"/>
-    <xacro:property name="calf_ixy" value="0.0"/>
-    <xacro:property name="calf_ixz" value="-0.000141163"/>
-    <xacro:property name="calf_iyy" value="0.003014022"/>
-    <xacro:property name="calf_iyz" value="0.0"/>
-    <xacro:property name="calf_izz" value="0.000032426"/>
-    <!-- foot -->
-    <xacro:property name="foot_mass" value="0.06"/>
 </robot>

File: quad_simulator/a1_description/xacro/leg.xacro (robot description, xacro)
@@ -42,8 +42,8 @@
             <dynamics damping="${damping}" friction="${friction}"/>
             <xacro:if value="${(mirror_dae == True)}">
-                <limit effort="${hip_torque_max}" velocity="${hip_velocity_max}" lower="${hip_min*PI/180.0}" upper="${hip_max*PI/180.0}"/>
+                <limit effort="${hip_torque_max}" velocity="${hip_velocity_max}" lower="${hip_position_min*PI/180.0}" upper="${hip_position_max*PI/180.0}"/>
             </xacro:if>
             <xacro:if value="${(mirror_dae == False)}">
-                <limit effort="${hip_torque_max}" velocity="${hip_velocity_max}" lower="${-hip_max*PI/180.0}" upper="${-hip_min*PI/180.0}"/>
+                <limit effort="${hip_torque_max}" velocity="${hip_velocity_max}" lower="${-hip_position_max*PI/180.0}" upper="${-hip_position_min*PI/180.0}"/>
             </xacro:if>
         </joint>
@@ -93,5 +93,5 @@
             <axis xyz="0 -1 0"/>
             <dynamics damping="${damping}" friction="${friction}"/>
-            <limit effort="${thigh_torque_max}" velocity="${thigh_velocity_max}" lower="${thigh_min*PI/180.0}" upper="${thigh_max*PI/180.0}"/>
+            <limit effort="${thigh_torque_max}" velocity="${thigh_velocity_max}" lower="${thigh_position_min*PI/180.0}" upper="${thigh_position_max*PI/180.0}"/>
         </joint>
         <link name="lower${suffix}">
@@ -121,5 +121,5 @@
             <axis xyz="0 1 0"/>
             <dynamics damping="${damping}" friction="${friction}"/>
-            <limit effort="${calf_torque_max}" velocity="${calf_velocity_max}" lower="${calf_min*PI/180.0}" upper="${calf_max*PI/180.0}"/>
+            <limit effort="${calf_torque_max}" velocity="${calf_velocity_max}" lower="${calf_position_min*PI/180.0}" upper="${calf_position_max*PI/180.0}"/>
         </joint>
         <link name="toe${suffix}">
